Commit message: Update bluerov_ros_playground: Modify launch files and add navigation improvements

File: model/BlueRov2.urdf.xacro (robot description, xacro)
@@ -11,5 +11,5 @@
         </joint>
         <link name="${name}">
-            <!--buoyancy><compensation>1.0</compensation></buoyancy>
+            <buoyancy><compensation>1.0</compensation></buoyancy>
             <visual name="${name}">
                 <geometry>
@@ -19,6 +19,6 @@
                     <color rgba="0 0 0 1"/>
                 </material>
-            </visual-->
-            <!--inertial>
+            </visual>
+            <inertial>
                 <mass value=".1"/>
                 <inertia
@@ -29,5 +29,5 @@
                     iyz="0.0"
                     izz=".1"/>
-                </inertial-->
+                </inertial>
             </link>
             <gazebo reference="${name}">
@@ -95,10 +95,10 @@
       izz="1"/>
     </inertial>
-    <!--collision>
+    <collision>
       <origin xyz="0 0 0" rpy="0 0 0"/>
       <geometry>
       <box size="0.5 0.5 0.5"/>
       </geometry>
-    </collision-->
+    </collision>
     <buoyancy>
         <compensation>0.2525</compensation>
@@ -119,5 +119,5 @@
   </link>
   <link name="camera_link">
-    <!-- visual>
+    <visual>
       <geometry>
         <box size="0.1 0.1 0.1"/>
@@ -126,5 +126,5 @@
         <color rgba="1 1 1 1"/>
       </material>
-    </visual -->
+    </visual>
   </link>
   <joint name="camera_joint" type="fixed">
